File: er-pass-mul.kicad_pcb (KiCad board)
At the start: 2 copper layers, 20 x 128.5 mm, 20 parts, among them J1 Input1, J2 Input2, J3 Output1, J4 Input3, J5 Input4, J6 Output2, J7 Input5, J8 Input6, J9 Output3

Commit message: removed cover
Parts:
- removed REF**: logo3, eurorack:logo3
- removed REF** (x9): mount_LUM_1502-03, eurorack:mount_LUM_1502-03
- removed REF**: cover_hp4_20mm, eurorack:cover_hp4_20mm
Other:
- board size 20 x 128.5 mm -> 15 x 105 mm
- board text removed: "MUL"
