File: er-pass-mul.kicad_pcb (KiCad board)
At the start: 2 copper layers, 20 x 128.5 mm, 20 parts, among them J1 Input1, J2 Input2, J3 Output1, J4 Input3, J5 Input4, J6 Output2, J7 Input5, J8 Input6, J9 Output3

Commit message: removed other panels
Parts:
- removed J1: Input1, eurorack:LUM 1502-03
- removed J2: Input2, eurorack:LUM 1502-03
- removed J3: Output1, eurorack:LUM 1502-03
- removed J4: Input3, eurorack:LUM 1502-03
- removed J5: Input4, eurorack:LUM 1502-03
- removed J6: Output2, eurorack:LUM 1502-03
- removed J7: Input5, eurorack:LUM 1502-03
- removed J8: Input6, eurorack:LUM 1502-03
- removed J9: Output3, eurorack:LUM 1502-03
Routing:
- net GND: track 120.1 -> 0.00 mm
- net Net-(J6-PadTN): track 51.2 -> 0.00 mm
- net Net-(J3-PadTN): track 43.6 -> 0.00 mm
- net Net-(J1-PadT): track 36.8 -> 0.00 mm
- removed copper zone on B.Cu, net GND
